File: X15-Pi-Shield.brd (EAGLE design)
At the start: 160 x 100 mm, 80 parts, among them J1 T2I, J2 T2I, J3 DF13-4P-1.25DSA, J4 T2I, J5 DF13-4P-1.25DSA, J6 DF13-4P-1.25DSA, Q1 220mA/50V/3.5Ω, Q2 2.5A/30V/105mΩ, Q3 220mA/50V/3.5Ω, Q4 220mA/50V/3.5Ω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

Commit message: hi
Parts:
- removed C3: 22nF, SparkFun-Capacitors:0603
- removed C5, C6: 0.1uF, SparkFun-Capacitors:0603
- removed D1: 250mA/100V, SparkFun-DiscreteSemi:SOD-323
- removed JP1: JUMPER-SMT_2_NO_SILK, SparkFun-Jumpers:SMT-JUMPER_2_NO_SILK
- removed R3, R5: 1k, SparkFun-Resistors:0603
- removed R4: 10k, SparkFun-Resistors:0603
- removed U$1: MAX3058, X15-Pi-Shield-Parts:SOIC-8(CHANGETHIS)]
- removed U$2: MCP2515, X15-Pi-Shield-Parts:SOIC-18
- R27, R28, R29, R30: value (none) -> 50k
Connections:
- removed net CAN_SILENT: JP1.1, U$1.8
- removed net N$17: U$6.4
- removed net N$18: U$6.5
- removed net N$19: U$6.6
- removed net N$20: U$6.7
- removed net N$4: C3.1, D1.A, R3.2, R4.1, R5.2
- removed net RESET: R3.1, U$2.17
- removed net RXCAN: U$1.4, U$2.2
- removed net TXCAN: U$1.1, U$2.1
- net 3V3: now also U$6.6; no longer C5.1, C6.1, D1.C, JP1.2, R4.2, U$1.3, U$2.18
- net CAN_H: no longer U$1.7
- net CAN_L: no longer U$1.6
- net CAN_RESET: no longer R5.1
- net CLK: no longer U$2.13
- net CS: no longer U$2.16
- net FAULT: no longer U$1.5
- net GND: no longer C3.2, C5.2, C6.2, U$1.2, U$2.9
- net INT: no longer U$2.12
- net MISO: no longer U$2.15
- net MOSI: no longer U$2.14
- net OSC1: no longer U$2.8
- net OSC2: no longer U$2.7
- net RX0_INT: now also U$6.4; no longer U$2.11
- net RX1_INT: now also U$6.5; no longer U$2.10

Commit message: Board Dimensions AGAIN
Other:
- board size 160 x 100 mm -> 69.8 x 73 mm
Changed lines of the file:
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@@
 <setting verticaltext="up"/>
 </settings>
-<grid distance="50" unitdist="mil" unit="mil" style="lines" multiple="1" display="no" altdistance="5" altunitdist="mil" altunit="mil"/>
+<grid distance="1" unitdist="mil" unit="mil" style="lines" multiple="1" display="no" altdistance="5" altunitdist="mil" altunit="mil"/>
 <layers>
 <layer number="1" name="Top" color="4" fill="1" visible="yes" active="yes"/>
@@
 <layer number="154" name="FabDoc2" color="7" fill="1" visible="yes" active="yes"/>
 <layer number="155" name="FabDoc3" color="7" fill="1" visible="yes" active="yes"/>
+<layer number="166" name="AntennaArea" color="7" fill="1" visible="yes" active="yes"/>
+<layer number="168" name="4mmHeightArea" color="7" fill="1" visible="yes" active="yes"/>
 <layer number="191" name="mNets" color="7" fill="1" visible="yes" active="yes"/>
 <layer number="192" name="mBusses" color="7" fill="1" visible="yes" active="yes"/>
@@
 <board>
 <plain>
-<wire x1="0" y1="0" x2="160" y2="0" width="0" layer="20"/>
-<wire x1="160" y1="0" x2="160" y2="100" width="0" layer="20"/>
-<wire x1="160" y1="100" x2="0" y2="100" width="0" layer="20"/>
-<wire x1="0" y1="100" x2="0" y2="0" width="0" layer="20"/>
+<wire x1="1.9812" y1="69.1388" x2="28.9052" y2="69.1388" width="0.1524" layer="20"/>
+<wire x1="28.9052" y1="69.1388" x2="29.7942" y2="70.0278" width="0.1524" layer="20" curve="90"/>
+<wire x1="29.7942" y1="70.0278" x2="29.7942" y2="72.0598" width="0.1524" layer="20"/>
+<wire x1="29.7942" y1="72.0598" x2="30.6832" y2="72.9488" width="0.1524" layer="20" curve="-90"/>
+<wire x1="30.6832" y1="72.9488" x2="68.0212" y2="72.9488" width="0.1524" layer="20"/>
+<wire x1="68.0212" y1="72.9488" x2="69.9262" y2="71.0438" width="0.1524" layer="20" curve="-90"/>
+<wire x1="69.9262" y1="71.0438" x2="69.9262" y2="1.8288" width="0.1524" layer="20"/>
+<wire x1="69.9262" y1="1.8288" x2="68.0212" y2="-0.0762" width="0.1524" layer="20" curve="-90"/>
+<wire x1="68.0212" y1="-0.0762" x2="1.9812" y2="-0.0762" width="0.1524" layer="20"/>
+<wire x1="1.9812" y1="-0.0762" x2="0.0762" y2="1.8288" width="0.1524" layer="20" curve="-90"/>
+<wire x1="0.0762" y1="1.8288" x2="0.0762" y2="67.2338" width="0.1524" layer="20"/>
+<wire x1="0.0762" y1="67.2338" x2="1.9812" y2="69.1388" width="0.1524" layer="20" curve="-90"/>
 </plain>
 <attributes>

Commit message: AAAAAAAAAAA
Parts:
- moved U$4 167.0 mm to (65.4, 4.09), turned to 90 degrees
- moved J11 163.6 mm to (66.6, 42.5), turned to 90 degrees
- moved J6 150.2 mm to (41.4, 49.5), turned to 180 degrees
- moved J5 142.7 mm to (50.2, 49.6), turned to 180 degrees
- moved J13 140.1 mm to (21.8, 29.7)
- moved J3 134.9 mm to (58.7, 49.4), turned to 180 degrees
- moved J7 134.7 mm to (4.70, 27.3), turned to 270 degrees
- moved J1 133.6 mm to (40.7, 65.6)
- moved U$6 131.1 mm to (20.5, 55.0), turned to 270 degrees
- moved C9 131.0 mm to (65.6, 34.3), turned to 270 degrees
- moved U$9 129.3 mm to (58.4, 8.94), turned to 180 degrees
- moved U$7 125.5 mm to (34.3, 5.46), turned to 90 degrees
- moved J2 125.5 mm to (7.21, 48.0), turned to 90 degrees
- moved J15 123.1 mm to (62.5, 45.1), turned to 270 degrees
- moved U$8 122.8 mm to (25.0, 7.14), turned to 180 degrees
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Routing:
- added copper zone on layer 1, net GND
- added copper zone on layer 16, net GND

Commit message: I'm slowly losing my mind
Parts:
- moved R25 173.7 mm to (47.1, 14.7), flipped to the bottom, turned to 180 degrees
- moved R24 168.3 mm to (47.0, 18.4), flipped to the bottom, turned to 180 degrees
- moved R26 168.3 mm to (37.3, 15.8), flipped to the bottom, turned to 270 degrees
- moved R22 165.8 mm to (45.2, 10.7), flipped to the bottom, turned to 180 degrees
- moved R23 156.8 mm to (37.2, 19.7), flipped to the bottom, turned to 90 degrees
- moved R30 155.9 mm to (24.1, 40.7), turned to 90 degrees
- moved R29 154.4 mm to (26.2, 40.8), turned to 90 degrees
- moved R28 152.8 mm to (28.2, 40.8), turned to 90 degrees
- moved R27 151.3 mm to (30.2, 40.9), turned to 90 degrees
- moved R21 150.4 mm to (24.9, 8.05), flipped to the bottom, turned to 270 degrees
- moved C11 148.4 mm to (16.6, 7.44), turned to 90 degrees
- moved R20 147.6 mm to (22.5, 6.27), flipped to the bottom, turned to 90 degrees
- moved C7 146.3 mm to (45.6, 37.2), flipped to the bottom, turned to 270 degrees
- moved C12 146.2 mm to (19.7, 17.8), flipped to the bottom
- moved C13 145.2 mm to (19.6, 23.7), flipped to the bottom, turned to 180 degrees
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Connections:
- net ROBOT_ARM: now also U$4.31
Routing:
- net 3V3: track 0.00 -> 222.8 mm, vias 0 -> 12
- net 5V: track 0.00 -> 220.1 mm, vias 0 -> 10
- net CAN_L: track 0.00 -> 179.1 mm, vias 0 -> 3
- net CAN_H: track 0.00 -> 169.3 mm, vias 0 -> 3
- net GPIO6: track 0.00 -> 141.5 mm, vias 0 -> 1
- net SDA: track 0.00 -> 131.6 mm, vias 0 -> 4
- net GPIO5: track 0.00 -> 128.0 mm, vias 0 -> 1
- net SCL: track 0.00 -> 127.5 mm, vias 0 -> 4
- net GPIO4: track 0.00 -> 112.2 mm, vias 0 -> 1
- net GPIO3: track 0.00 -> 104.0 mm, vias 0 -> 1
- net GPIO2: track 0.00 -> 98.8 mm, vias 0 -> 1
- net GPIO1: track 0.00 -> 88.3 mm, vias 0 -> 1
- net ROBOT_ARM: track 0.00 -> 86.3 mm, vias 0 -> 8
- net A_INT: track 0.00 -> 63.5 mm, vias 0 -> 1
- net IMU_INT: track 0.00 -> 51.7 mm, vias 0 -> 3
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
Commit message: Hi Katherine
Parts:
- removed J1, J2, J4: T2I, X15-Pi-Shield-Parts:T2I
- removed U1: ULN2003AD, X15-Pi-Shield-Parts:16-SOIC
- moved R30 1.23 mm to (23.4, 41.8)
Connections:
- removed net DI1: J2.2, U$4.36
- removed net DI2: J2.3, U$4.38
- removed net PWM: U$4.33
- removed net SOL1_1: U$9.1, U1.16
- removed net SOL2_1: U$9.3, U1.15
- removed net SOL3_1: U$9.5, U1.14
- removed net SOL4_1: U$9.7, U1.13
- removed net SOL5_1: U$9.9, U1.12
- removed net SOL6_1: U$9.11, U1.11
- new net ROBOT_ARM_2: U$4.33, U$9.16
- net 12V: no longer U1.9
- net 5V: no longer J2.1
- net CAN_H: no longer J1.2, J4.2
- net CAN_L: no longer J1.3, J4.3
- net GND: no longer J2.4, U1.8
- net GPIO1: now also U$4.36, U$9.1; no longer U$4.12, U1.1
- net GPIO2: now also U$9.3; no longer U1.2
- net GPIO3: now also U$9.5; no longer U1.3
- net GPIO4: now also U$9.7; no longer U1.4
- net GPIO5: now also U$4.38, U$9.9; no longer U$4.32, U1.5
- net GPIO6: now also U$9.11; no longer U1.6
- net ROBOT_ARM: now also U$4.32; no longer U$4.31
Routing:
- net GND: track 35.7 -> 265.0 mm, vias 4 -> 27
- net ROBOT_ARM_2: track 0.00 -> 68.5 mm, vias 0 -> 7
- net GPIO6: track 141.5 -> 97.7 mm, vias 1 -> 0
- net GPIO3: track 104.0 -> 67.5 mm, vias 1 -> 8
- net GPIO5: track 128.0 -> 101.2 mm
- net SOL6_1: track 22.6 -> 0.00 mm
- net SOL5_1: track 20.2 -> 0.00 mm
- net GPIO4: track 112.2 -> 93.6 mm, vias 1 -> 5
- net SOL4_1: track 17.6 -> 0.00 mm
- net SOL3_1: track 15.0 -> 0.00 mm
- net GPIO1: track 88.3 -> 102.8 mm, vias 1 -> 2
- net 5V: track 220.1 -> 207.3 mm
- net SOL2_1: track 12.6 -> 0.00 mm
- net SOL1_1: track 9.65 -> 0.00 mm
- net DI1: track 8.28 -> 0.00 mm
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
Commit message: r/RoastMe
Parts:
- moved C4 0.83 mm to (18.0, 34.6)
- moved R2 0.33 mm to (27.1, 58.2)
- moved C2 0.05 mm to (25.9, 62.0)
Routing:
- net GPIO2: track 104.1 -> 108.6 mm
- net GPIO1: track 102.8 -> 107.0 mm
- net N$2: track 5.27 -> 8.20 mm
- net GPIO5: track 101.2 -> 103.6 mm
- net GND: track 265.0 -> 267.2 mm
- net CAN_RESET: track 32.6 -> 34.6 mm
- net IMU_RESET: track 28.5 -> 30.3 mm
- net GPIO4: track 93.6 -> 95.1 mm
- net GPIO6: track 97.7 -> 99.1 mm
- net N$3: track 5.73 -> 7.11 mm
- net ROBOT_ARM: track 84.5 -> 83.2 mm
- net CAN_H: track 169.2 -> 170.4 mm
- net ROBOT_ARM_2: track 68.5 -> 69.6 mm
- net IMU_INT: track 51.8 -> 52.9 mm
- net CLK: track 29.2 -> 30.1 mm
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
Commit message: I swear its good this time
Routing:
- net SDA: track 132.3 -> 137.7 mm, vias 4 -> 6
- net !AMP_RESET: track 51.6 -> 54.4 mm
- net IMU_INT: track 52.9 -> 55.4 mm
- net 3V3: track 222.6 -> 224.2 mm
- net CS: track 35.5 -> 36.8 mm
- net MOSI: track 51.5 -> 52.8 mm
- net SCL: track 128.1 -> 129.3 mm
- net 5V: track 207.6 -> 208.7 mm
- net ROBOT_ARM_2: track 69.6 -> 70.4 mm
- net MISO: track 43.8 -> 44.5 mm
- net CAN_L: track 179.0 -> 178.9 mm, vias 4 -> 2
- net CAN_H: track 170.4 -> 170.3 mm, vias 4 -> 2

Commit message: AAAAAAAAAAAAAAAAAAAAAAAAAAA
Routing:
- net GND: track 267.4 -> 294.5 mm, vias 27 -> 30
Changed lines of the file:
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@@
 <wire x1="17.0688" y1="20.9296" x2="17.6276" y2="21.4884" width="0.254" layer="1"/>
 <wire x1="18.161" y1="22.7838" x2="21.8694" y2="22.7838" width="0.254" layer="1"/>
-<wire x1="11.6586" y1="35.306" x2="14.1986" y2="42.926" width="0" layer="19" extent="1-1"/>
+<wire x1="11.6586" y1="35.306" x2="8.9408" y2="35.306" width="0.254" layer="16"/>
+<wire x1="8.9408" y1="35.306" x2="8.509" y2="35.7378" width="0.254" layer="16"/>
+<via x="8.509" y="35.7378" extent="1-16" drill="0.35"/>
+<wire x1="8.509" y1="35.7378" x2="5.9436" y2="35.7378" width="0.254" layer="1"/>
+<wire x1="5.9436" y1="35.7378" x2="5.8956" y2="35.7858" width="0.254" layer="1"/>
+<wire x1="5.8956" y1="38.1508" x2="5.8956" y2="35.7858" width="0.254" layer="1"/>
+<wire x1="5.8956" y1="38.1508" x2="5.6416" y2="38.4048" width="0.254" layer="1"/>
+<via x="5.6416" y="38.4048" extent="1-16" drill="0.35"/>
+<wire x1="5.6416" y1="38.4048" x2="5.6416" y2="39.2656" width="0.254" layer="16"/>
+<wire x1="5.6416" y1="39.2656" x2="3.6068" y2="41.3004" width="0.254" layer="16"/>
+<via x="3.6068" y="41.3004" extent="1-16" drill="0.35"/>
+<wire x1="3.6068" y1="41.3004" x2="3.6068" y2="47.2694" width="0.254" layer="1"/>
+<wire x1="3.6068" y1="47.2694" x2="4.7752" y2="48.4378" width="0.254" layer="1"/>
+<wire x1="4.7752" y1="48.4378" x2="10.033" y2="48.4378" width="0.254" layer="1"/>
+<wire x1="10.033" y1="48.4378" x2="10.4902" y2="47.9806" width="0.254" layer="1"/>
+<wire x1="10.4902" y1="47.9806" x2="11.6332" y2="47.9806" width="0.254" layer="1"/>
+<wire x1="11.6332" y1="47.9806" x2="11.6586" y2="48.006" width="0.254" layer="1"/>
 </signal>
 <signal name="N$1">
@@
 <wire x1="21.4884" y1="10.4394" x2="22.5298" y2="9.398" width="0.762" layer="1"/>
 <via x="22.5298" y="9.398" extent="1-16" drill="0.85"/>
-<wire x1="22.5044" y1="7.1746" x2="22.4536" y2="7.1238" width="0.762" layer="16"/>
 <wire x1="22.5298" y1="9.398" x2="24.0284" y2="7.8994" width="0.762" layer="1"/>
 <wire x1="24.0284" y1="7.8994" x2="26.5684" y2="7.8994" width="0.762" layer="1"/>
@@
 <wire x1="66.6242" y1="64.3636" x2="58.42" y2="56.1594" width="0.254" layer="16"/>
 <wire x1="58.42" y1="56.1594" x2="54.2798" y2="56.1594" width="0.254" layer="16"/>
-<wire x1="45.847" y1="69.8754" x2="45.8216" y2="69.85" width="0.254" layer="16"/>
 <wire x1="35.9156" y1="59.944" x2="45.8216" y2="69.85" width="0.254" layer="16"/>
 <wire x1="35.9156" y1="59.944" x2="32.004" y2="59.944" width="0.254" layer="16"/>
@@
 <wire x1="20.4978" y1="43.6372" x2="20.4978" y2="45.591" width="0.254" layer="1"/>
 <wire x1="20.4978" y1="45.591" x2="20.447" y2="45.6418" width="0.254" layer="1"/>
-<wire x1="45.8216" y1="69.85" x2="49.2252" y2="69.85" width="0.254" layer="16"/>
 <wire x1="49.2252" y1="69.85" x2="50.7492" y2="68.326" width="0.254" layer="16"/>
 <wire x1="50.7492" y1="68.326" x2="50.7492" y2="59.7084" width="0.254" layer="16"/>
 <wire x1="50.7492" y1="59.7084" x2="50.74" y2="59.6992" width="0.254" layer="16"/>
+<wire x1="45.8216" y1="69.85" x2="49.2252" y2="69.85" width="0.254" layer="16"/>
 </signal>
 <signal name="CAN_L">
@@
 <via x="32.1818" y="13.1826" extent="1-16" drill="0.35"/>
 <wire x1="15.7734" y1="13.89925" x2="16.284125" y2="13.388525" width="0.254" layer="16"/>
-<wire x1="16.284125" y1="13.388525" x2="16.36025" y2="13.3124" width="0.254" layer="16"/>
 <wire x1="15.7734" y1="13.89925" x2="15.7734" y2="15.367" width="0.254" layer="16"/>
 <wire x1="16.0274" y1="18.8722" x2="16.024675" y2="18.874925" width="0.1524" layer="16"/>
@@
 <wire x1="37.6428" y1="5.1308" x2="37.338" y2="5.4356" width="0.254" layer="16"/>
 <wire x1="37.338" y1="5.4356" x2="37.338" y2="8.5598" width="0.254" layer="16"/>
-<wire x1="37.338" y1="8.5598" x2="37.7444" y2="8.9662" width="0.254" layer="16"/>
-<wire x1="37.7444" y1="8.9662" x2="40.1574" y2="8.9662" width="0.254" layer="16"/>
-<wire x1="40.1574" y1="8.9662" x2="40.6908" y2="9.4996" width="0.254" layer="16"/>
+<wire x1="37.338" y1="8.5598" x2="37.8206" y2="9.0424" width="0.254" layer="16"/>
+<wire x1="37.8206" y1="9.0424" x2="40.2336" y2="9.0424" width="0.254" layer="16"/>
+<wire x1="40.2336" y1="9.0424" x2="40.6908" y2="9.4996" width="0.254" layer="16"/>
 <wire x1="40.6908" y1="9.4996" x2="40.6908" y2="9.5758" width="0.1524" layer="16"/>
 <via x="40.6908" y="9.5758" extent="1-16" drill="0.35"/>
@@
 <wire x1="40.132" y1="19.9898" x2="40.132" y2="16.256" width="0.254" layer="1"/>
 <wire x1="40.132" y1="16.256" x2="42.545" y2="13.843" width="0.254" layer="1"/>
-<wire x1="40.6583875" y1="8.6134" x2="38.7124" y2="8.6134" width="0.254" layer="1"/>
-<wire x1="38.5826" y1="8.4836" x2="38.5826" y2="7.6708" width="0.254" layer="1"/>
+<wire x1="38.5826" y1="7.6708" x2="38.5826" y2="8.4836" width="0.254" layer="1"/>
 <wire x1="32.893" y1="45.212" x2="33.4264" y2="44.6786" width="0.254" layer="1"/>
 <wire x1="35.6362" y1="27.051" x2="38.1762" y2="24.511" width="0.254" layer="1"/>
-<wire x1="38.7124" y1="8.6134" x2="38.5826" y2="8.4836" width="0.254" layer="1"/>
 <wire x1="33.4264" y1="38.9636" x2="33.8836" y2="38.5064" width="0.254" layer="1"/>
 <wire x1="33.8836" y1="35.7124" x2="33.4264" y2="35.2552" width="0.254" layer="1"/>
@@
 <wire x1="33.4264" y1="44.6786" x2="33.4264" y2="38.9636" width="0.254" layer="1"/>
 <wire x1="33.8836" y1="38.5064" x2="33.8836" y2="35.7124" width="0.254" layer="1"/>
-<wire x1="42.545" y1="9.2202" x2="41.9608" y2="8.636" width="0.254" layer="1"/>
-<wire x1="41.5539625" y1="8.7122" x2="40.6912375" y2="8.7122" width="0.254" layer="1"/>
-<wire x1="40.6912375" y1="8.7122" x2="40.6254125" y2="8.646375" width="0.254" layer="1"/>
-<wire x1="41.9608" y1="8.636" x2="41.6301625" y2="8.636" width="0.254" layer="1"/>
-<wire x1="41.6301625" y1="8.636" x2="41.5539625" y2="8.7122" width="0.254" layer="1"/>
-<wire x1="42.545" y1="13.843" x2="42.545" y2="9.2202" width="0.254" layer="1"/>
-<wire x1="40.6254125" y1="8.646375" x2="40.6583875" y2="8.6134" width="0" layer="19" extent="1-1"/>
+<wire x1="42.545" y1="9.2202" x2="42.545" y2="13.843" width="0.254" layer="1"/>
+<wire x1="40.6658375" y1="8.6868" x2="40.6912375" y2="8.7122" width="0.254" layer="1"/>
+<wire x1="42.037" y1="8.7122" x2="42.545" y2="9.2202" width="0.254" layer="1"/>
+<wire x1="40.6912375" y1="8.7122" x2="42.037" y2="8.7122" width="0.254" layer="1"/>
+<wire x1="38.5826" y1="8.4836" x2="38.7858" y2="8.6868" width="0.254" layer="1"/>
+<wire x1="38.7858" y1="8.6868" x2="40.6658375" y2="8.6868" width="0.254" layer="1"/>
 </signal>
 </signals>
