File: X15-Pi-Shield.brd (EAGLE design)
At the start: 69.8 x 73 mm, 66 parts, among them J3 DF13-4P-1.25DSA, J5 DF13-4P-1.25DSA, J6 DF13-4P-1.25DSA, Q1 220mA/50V/3.5Ω, Q2 2.5A/30V/105mΩ, Q3 220mA/50V/3.5Ω, Q4 220mA/50V/3.5Ω, Q5 220mA/50V/3.5Ω, U2 MAX1136EUA-T, Y2 ECS-80-S-4X

Commit message: AAAA
Parts:
- removed C9: 47uF, SparkFun-Capacitors:PANASONIC_D
- moved C10 0.22 mm to (16.7, 11.3)
Connections:
- removed net 12V: C9.+, U$9.2, U$9.4
- net GND: no longer C9.-
Routing:
- net 12V: track 31.3 -> 0.00 mm
- net GND: track 294.5 -> 310.7 mm, vias 30 -> 31
- net SDA: track 137.7 -> 151.2 mm, vias 6 -> 7
- net CAN_L: track 178.9 -> 171.8 mm
- net TX: track 15.1 -> 16.8 mm
- net GPIO1: track 107.0 -> 108.3 mm
- net RX: track 14.9 -> 16.2 mm
- net SCL: track 129.3 -> 130.3 mm
- net CAN_H: track 170.3 -> 171.0 mm, vias 2 -> 1
- net !AMP_RESET: track 54.3 -> 54.9 mm
- net 3V3: vias 12 -> 11

Commit message: HI :D
Parts:
- removed D2: 250mA/100V, SparkFun-DiscreteSemi:SOD-323
- removed Q1: 220mA/50V/3.5Ω, SparkFun-DiscreteSemi:SOT23-3
- removed R6: 470, SparkFun-Resistors:0603
- removed R7: 68, SparkFun-Resistors:0603
- renumbered D3 to 5V, D4 to 3V, D5 to OVERCURRENT
Connections:
- removed net FAULT: Q1.1, R6.2
- removed net N$5: D2.C, Q1.3
- removed net N$6: D2.A, R7.1
- net 3V3: no longer R6.1, R7.2
- net GND: no longer Q1.2
Routing:
- net 3V3: track 224.2 -> 194.8 mm, vias 11 -> 9
- net FAULT: track 6.96 -> 0.00 mm, vias 1 -> 0
- net N$5: track 3.32 -> 0.00 mm
- net N$6: track 2.55 -> 0.00 mm
