File: X15-Pi-Shield.sch (EAGLE design)
At the start: 70 parts, among them J1 T2I, J2 T2I, J3 DF13-4P-1.25DSA, J4 T2I, J5 DF13-4P-1.25DSA, J6 DF13-4P-1.25DSA, Q1 220mA/50V/3.5Ω, Q2 2.5A/30V/105mΩ, Q3 220mA/50V/3.5Ω, Q4 220mA/50V/3.5Ω, Q5 220mA/50V/3.5Ω, U1 ULN2003AD, U2 MAX1136EUA-T, Y2 ECS-80-S-4X

Commit message: Hi Katherine
Parts:
- removed J1, J2, J4: T2I, X15-Pi-Shield-Parts:T2I
- removed U1: ULN2003AD, X15-Pi-Shield-Parts:ULN2003AD
Connections:
- removed net DI1: J2.2, U$4.GPIO16
- removed net DI2: J2.3, U$4.GPIO20
- removed net PWM: U$4.GPIO13
- removed net SOL1_1: U$9.14, U1.OUT1
- removed net SOL2_1: U$9.16, U1.OUT2
- removed net SOL3_1: U$9.18, U1.OUT3
- removed net SOL4_1: U$9.20, U1.OUT4
- removed net SOL5_1: U$9.22, U1.OUT5
- removed net SOL6_1: U$9.24, U1.OUT6
- new net ROBOT_ARM_2: U$4.GPIO13, U$9.3
- net 12V: no longer U1.COM
- net 5V: no longer J2.1
- net CAN_H: no longer J1.2, J4.2
- net CAN_L: no longer J1.3, J4.3
- net GND: no longer J2.4, U1.GND
- net GPIO1: now also U$4.GPIO16, U$9.14; no longer U$4.GPIO18, U1.IN1
- net GPIO2: now also U$9.16; no longer U1.IN2
- net GPIO3: now also U$9.18; no longer U1.IN3
- net GPIO4: now also U$9.20; no longer U1.IN4
- net GPIO5: now also U$4.GPIO20, U$9.22; no longer U$4.GPIO12, U1.IN5
- net GPIO6: now also U$9.24; no longer U1.IN6
- net ROBOT_ARM: now also U$4.GPIO12; no longer U$4.GPIO6
Other:
- note added: "PINS 15/16 is a new addition for PWM signals to the robot arm"
- note removed: "NPN Array"
- note removed: "PIN 15 is a new addition for PWM signal to the robot arm"

Commit message: ASAIDFNODIWBEOIYBF
Parts:
- removed C9: 47uF, SparkFun-Capacitors:47UF-POLAR-PANASONIC_D-35V-20%
Connections:
- removed net 12V: C9.+, U$9.13, U$9.15
- net GND: no longer C9.-
Other:
- note removed: "UZ476M035HEHTA decoupling cap for solenoids"
Changed lines of the file:
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@@
 <part name="GND29" library="SparkFun-PowerSymbols" library_urn="urn:adsk.eagle:library:530" deviceset="GND" device=""/>
 <part name="FRAME4" library="SparkFun-Aesthetics" library_urn="urn:adsk.eagle:library:507" deviceset="FRAME-A4L" device=""/>
-<part name="C9" library="SparkFun-Capacitors" library_urn="urn:adsk.eagle:library:510" deviceset="47UF-POLAR" device="-PANASONIC_D-35V-20%" package3d_urn="urn:adsk.eagle:package:37420/1" value="47uF"/>
 <part name="D3" library="SparkFun-LED" library_urn="urn:adsk.eagle:library:529" deviceset="LED" device="0603" package3d_urn="urn:adsk.eagle:package:39354/1"/>
 <part name="D4" library="SparkFun-LED" library_urn="urn:adsk.eagle:library:529" deviceset="LED" device="0603" package3d_urn="urn:adsk.eagle:package:39354/1"/>
@@
 <part name="C13" library="SparkFun-Capacitors" library_urn="urn:adsk.eagle:library:510" deviceset="0.1UF" device="-0603-25V-(+80/-20%)" package3d_urn="urn:adsk.eagle:package:37414/1" value="0.1uF"/>
 <part name="GND36" library="SparkFun-PowerSymbols" library_urn="urn:adsk.eagle:library:530" deviceset="GND" device=""/>
-<part name="GND38" library="SparkFun-PowerSymbols" library_urn="urn:adsk.eagle:library:530" deviceset="GND" device=""/>
 <part name="GND39" library="SparkFun-PowerSymbols" library_urn="urn:adsk.eagle:library:530" deviceset="GND" device=""/>
 <part name="GND40" library="SparkFun-PowerSymbols" library_urn="urn:adsk.eagle:library:530" deviceset="GND" device=""/>
@@
 <plain>
 <text x="198.12" y="160.02" size="1.778" layer="91">Connectors</text>
-<text x="53.34" y="73.66" size="1.778" layer="91">UZ476M035HEHTA
-decoupling cap for solenoids</text>
 <text x="187.96" y="121.92" size="1.778" layer="91">PINS 15/16 is a new addition for PWM
 signals to the robot arm</text>
@@
 <attribute name="SHEET" x="195.58" y="1.27" size="2.54" layer="94" font="vector"/>
 </instance>
-<instance part="C9" gate="G$1" x="88.9" y="73.66" smashed="yes">
-<attribute name="NAME" x="89.916" y="74.295" size="1.778" layer="95" font="vector"/>
-<attribute name="VALUE" x="89.916" y="69.469" size="1.778" layer="96" font="vector"/>
-</instance>
-<instance part="GND38" gate="1" x="88.9" y="60.96" smashed="yes">
-<attribute name="VALUE" x="88.9" y="60.706" size="1.778" layer="96" align="top-center"/>
-</instance>
 <instance part="U$9" gate="G$1" x="203.2" y="144.78" smashed="yes">
 <attribute name="NAME" x="198.755" y="154.305" size="1.778" layer="95" font="vector"/>
@@
 </busses>
 <nets>
-<net name="12V" class="0">
-<segment>
-<wire x1="195.58" y1="151.13" x2="182.88" y2="151.13" width="0.1524" layer="91"/>
-<label x="185.42" y="151.13" size="1.778" layer="95"/>
-<pinref part="U$9" gate="G$1" pin="13"/>
-</segment>
-<segment>
-<wire x1="195.58" y1="148.59" x2="182.88" y2="148.59" width="0.1524" layer="91"/>
-<label x="185.42" y="148.59" size="1.778" layer="95"/>
-<pinref part="U$9" gate="G$1" pin="15"/>
-</segment>
-<segment>
-<pinref part="C9" gate="G$1" pin="+"/>
-<wire x1="88.9" y1="76.2" x2="88.9" y2="81.28" width="0.1524" layer="91"/>
-<label x="88.9" y="81.28" size="1.778" layer="95"/>
-</segment>
-</net>
 <net name="GND" class="0">
 <segment>
@@
 <pinref part="U$9" gate="G$1" pin="21"/>
 </segment>
-<segment>
-<pinref part="C9" gate="G$1" pin="-"/>
-<wire x1="88.9" y1="68.58" x2="88.9" y2="63.5" width="0.1524" layer="91"/>
-<pinref part="GND38" gate="1" pin="GND"/>
-</segment>
-</net>
+</net>

Commit message: HI :D
Parts:
- removed D2: 250mA/100V, SparkFun-DiscreteSemi:DIODE-BAS16J
- removed Q1: 220mA/50V/3.5Ω, SparkFun-DiscreteSemi:MOSFET-NCH-BSS138
- removed R6: 470, SparkFun-Resistors:RESISTOR0603
- removed R7: 68, SparkFun-Resistors:RESISTOR0603
- renumbered D3 to 5V, D4 to 3V, D5 to OVERCURRENT
Connections:
- removed net FAULT: Q1.G, R6.2
- removed net N$5: D2.C, Q1.D
- removed net N$6: D2.A, R7.1
- net 3V3: no longer R6.1, R7.2
- net GND: no longer Q1.S
Other:
- note removed: "IS THIS NEEDED ANYMORE??? FAULT NOT CONNECTED TO ANYTHING"
- note removed: "LED turns on when CAN Tranceiver detects a fault"
